File: brainboardV1.0/MESC_brain_board.kicad_sch (KiCad schematic)
At the start: 17 parts, among them J1 Conn_01x18, J2 Conn_01x04, Q1 my_BC337, U2 TJA1050T/CM,118, U2 Teensy4.0

Commit message: minor changes
Other:
- note added: "3.3V CAN transcievers only"
Changed lines of the file:
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@@
+		)
+	)
+	(text "3.3V CAN transcievers only"
+		(exclude_from_sim no)
+		(at 52.07 73.66 0)
+		(effects
+			(font
+				(size 1.27 1.27)
+			)
 		)
 	)
