Commit message: modeling scripts

File: modeling/pendulum.urdf (robot description, URDF)
Before this commit: robot pendulum, 2 links, 1 joints
Links:
- link pendulum_link: mass 1.4954147111892706 -> 0.18269208799931075
Joints:
- joint hinge: origin xyz=0.0 0.0 0.05 rpy=0 0 0 -> xyz=-1.6047283079967634e-18 0.00969999999998872 0.4 rpy=0 0 0
