File: brainboardV1.2/MESC_brain_board.kicad_pcb (KiCad board)
At the start: 4 copper layers, 90.5 x 68.6 mm, 57 parts, among them J1 Conn_01x18, J12 Conn_01x03, J13 Conn_01x03, J14 SERIAL1, J15 Conn_01x03, J22 Conn_01x01, J24 Conn_01x01, J25 Conn_01x01, Q1 my_BC337, U1 TJA1050T/CM,118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

Commit message: finalizing brain board v1.2
Parts:
- removed 20k_3: 20k, Resistor_SMD:R_0603_1608Metric
- removed C24, C26, C28, C29: 10uF, Capacitor_SMD:C_0603_1608Metric
- removed D23: BZG03C15, Diode_SMD:D_SMA
- removed D_BLU1: LED BLU, LED_SMD:LED_0603_1608Metric
- removed MESC2: Conn_01x06, Connector_JST:JST_PH_B6B-PH-K_1x06_P2.00mm_Vertical
- removed MP1: Conn_01x08, Connector_PinSocket_2.54mm:PinSocket_1x08_P2.54mm_Vertical
- removed the REF** at (108.3, 74.8)
- removed the REF** at (161.3, 35.7)
- removed Tp12V21: 12V Pad, TestPoint:TestPoint_THTPad_D2.0mm_Drill1.0mm
- added 20k_21: 20k, Resistor_SMD:R_0603_1608Metric, F.Cu at (74.4, 63.9)
- added C21: 100nF, Capacitor_SMD:C_0805_2012Metric, F.Cu at (68.5, 68.4)
- added D_BLU21: LED BLU, LED_SMD:LED_0603_1608Metric, F.Cu at (74.4, 62.2)
- added J21: Conn_01x07, Connector_JST:JST_PH_B7B-PH-K_1x07_P2.00mm_Vertical, F.Cu at (23.2, 54.2)
- added REF**: MountingHole_3.2mm_M3, MountingHole:MountingHole_3.2mm_M3, F.Cu at (23.4, 13.3)
- added REF**: MountingHole_3.2mm_M3, MountingHole:MountingHole_3.2mm_M3, F.Cu at (79.8, 13.3)
- added U21: LD1117S18TR_SOT223, Package_TO_SOT_SMD:SOT-223-3_TabPin2, F.Cu at (72.6, 57.1)
- C23: value 100nF -> C_Polarized_Small_US; footprint Capacitor_SMD:C_0805_2012Metric -> Capacitor_Tantalum_SMD:CP_EIA-3216-18_Kemet-A
- C25, C27: footprint Capacitor_SMD:C_0603_1608Metric -> Capacitor_SMD:C_0805_2012Metric
- moved REF** 144.6 mm to (23.4, 89.9)
- moved REF** 85.3 mm to (79.8, 89.9)
- moved C27 73.9 mm to (71.7, 63.0), turned to -90 degrees
- moved C25 73.8 mm to (69.5, 63.0), turned to -90 degrees
- moved C23 59.7 mm to (77.7, 53.8)
- moved J22 45.4 mm to (66.5, 52.5)
- moved J24 39.1 mm to (79.5, 59.1), turned to 90 degrees
- moved J25 31.5 mm to (79.5, 64.7), turned to 90 degrees
- moved Q1 27.3 mm to (54.3, 67.0), turned to -90 degrees
- moved 5k_2 23.3 mm to (24.4, 36.1), turned to 90 degrees
- moved 1k_1 22.7 mm to (57.4, 66.8)
- moved LS1 22.4 mm to (59.9, 76.6), turned to 180 degrees
- moved U24 21.8 mm to (76.5, 70.2), turned to 180 degrees
- moved 10k_1 20.0 mm to (59.7, 48.5)
- moved 10k_4 20.0 mm to (79.1, 50.3)
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Connections:
- C23 pad 1: VBAT -> +3.3V
- MESC1 pad 3: PB6_1 -> GPIO1
- MESC1 pad 4: PB5_1 -> GPIO2
- MESC1 pad 5: PB4_1 -> GPIO3
- MESC1 pad 6: PB3_1 -> GPIO4
- U2 pad 12: PB3_1 -> CS
- U2 pad 13: PB4_1 -> MOSI
- U2 pad 14: PB5_1 -> MISO
- U2 pad 20: SPEAKER -> SCLK
- U2 pad 21: PB3_2 -> SPEAKER
- U2 pad 22: PB4_2 -> GPIO4
- U2 pad 23: PB5_2 -> GPIO3
- U2 pad 24: BUTTON -> GPIO2
- U2 pad 25: /MPU6050_SDA -> GPIO1
- U2 pad 26: /MPU6050_SCL -> BUTTON
- U2 pad 27: unconnected-(U2-20_A6_TX5_LRCLK1-Pad27) -> INT1
- U2 pad 28: VSENSE -> unconnected-(U2-21_A7_RX5_BCLK1-Pad28)
- U24 pad 1: +12V -> Vcc
Routing:
- net +5V: track 71.5 -> 304.2 mm
- net BUTTON: track 11.7 -> 78.4 mm, vias 0 -> 1
- net RC_Z: track 0.00 -> 59.9 mm
- net RC_Y: track 0.00 -> 54.4 mm
- net RC_X: track 0.00 -> 49.4 mm
- net RC_Mode: track 0.00 -> 45.7 mm
- net VSENSE: track 40.9 -> 0.00 mm, vias 2 -> 0
- net SPEAKER: track 0.00 -> 25.7 mm, vias 0 -> 1
- net INT1: track 0.00 -> 24.8 mm, vias 0 -> 1
- net RC_Steering: track 0.00 -> 23.8 mm
- net RC_Throttle: track 14.8 -> 37.2 mm
- net SCLK: track 0.00 -> 22.3 mm
- net +3.3V: track 12.7 -> 33.5 mm, vias 6 -> 8
- net Vcc: track 0.00 -> 17.7 mm
- net unconnected-(U2-21_A7_RX5_BCLK1-Pad28): track 0.00 -> 16.0 mm, vias 0 -> 1
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Other:
- board size 90.5 x 68.6 mm -> 64 x 84.5 mm
- board text removed: "MESC1"
- board text removed: "MESC2"
- board text removed: "PB3"
- board text removed: "PB4"
- board text removed: "PB5"

Commit message: documentation stuff
Parts:
- added J23: Conn_01x01, Connector_PinSocket_2.54mm:PinSocket_1x01_P2.54mm_Vertical, F.Cu at (45.5, 62.8)
- moved REF** 74.1 mm to (96.7, 23.7), turned to -90 degrees
- moved REF** 68.9 mm to (96.7, 80.1), turned to -90 degrees
- moved REF** 66.3 mm to (20.1, 23.7), turned to -90 degrees
- moved 20k_1 62.8 mm to (87.1, 24.7), turned to 180 degrees
- moved REF** 60.5 mm to (20.1, 80.1), turned to -90 degrees
- moved D_RED1 59.3 mm to (83.7, 24.8), turned to 180 degrees
- moved D_GRN1 53.4 mm to (77.1, 24.7), turned to 0 degrees
- moved 10k_8 51.3 mm to (29.1, 80.7), turned to 0 degrees
- moved 5k_2 50.9 mm to (73.9, 24.7), turned to 0 degrees
- moved S1 46.1 mm to (29.0, 75.1), turned to -90 degrees
- moved J21 44.8 mm to (55.8, 23.5), turned to 0 degrees
- moved J1 41.9 mm to (43.0, 28.0), turned to -90 degrees
- moved DC_1 41.9 mm to (29.0, 69.6), turned to 180 degrees
- moved J14 40.8 mm to (64.8, 77.1), turned to 90 degrees
- moved J13 39.6 mm to (67.1, 69.4), turned to 180 degrees
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Routing:
- net +5V: track 304.2 -> 278.2 mm
- net Net-(J14-Pin_1): track 18.1 -> 37.0 mm
- net unconnected-(U2-21_A7_RX5_BCLK1-Pad28): track 16.0 -> 0.00 mm, vias 1 -> 0
- net ESP_RX_OUT: track 10.5 -> 18.2 mm
- net U0RXD: track 27.6 -> 20.3 mm
- net /CAN_TX: track 29.8 -> 23.1 mm
- net ESP_TX: track 55.9 -> 61.0 mm, vias 0 -> 1
- net U0TXD: track 24.9 -> 20.7 mm
- net Net-(D_BLU2-A): track 7.14 -> 4.64 mm
- net ESP_EN: track 28.3 -> 30.6 mm
- net IO0: track 14.1 -> 15.6 mm
- net ESP_TX_OUT: track 10.4 -> 8.88 mm
- net /CAN_RX: track 33.1 -> 32.0 mm
- net Net-(J13-Pin_2): track 5.03 -> 4.26 mm
- net Net-(J12-Pin_2): track 3.64 -> 4.26 mm
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Other:
- board size 64 x 84.5 mm -> 84.5 x 64 mm
- board text removed: "ESP32 PROG"
- board text removed: "ESP32 PROG VOLT SELECT"
