File: brainboardV1.2/MESC_brain_board.kicad_sch (KiCad schematic)
At the start: 17 parts, among them J1 Conn_01x18, J2 Conn_01x04, Q1 my_BC337, U2 TJA1050T/CM,118, U2 Teensy4.0

Commit message: finalizing brain board v1.2
Parts:
- removed MESC2: Conn_01x06, Connector_JST:JST_PH_B6B-PH-K_1x06_P2.00mm_Vertical, symbol Connector_Generic:Conn_01x06
- removed MP1: Conn_01x08, Connector_PinSocket_2.54mm:PinSocket_1x08_P2.54mm_Vertical, symbol Connector_Generic:Conn_01x08
- added J21: Conn_01x07, Connector_JST:JST_PH_B7B-PH-K_1x07_P2.00mm_Vertical, symbol Connector_Generic:Conn_01x07
Connections:
- net MPU6050_SCL is gone; now on net BUTTON: U2.26 (19_A5_SCL0)
- net PB3_2 is gone; now on net SPEAKER: U2.21 (14_A0_TX3_SPDIF_OUT)
- net PB5_2 is gone; now on net GPIO3: U2.23 (16_A2_RX4_SCL1)
- net PB6_1 is gone; now on net GPIO1: MESC1.3 (Pin_3)
- net +3.3V: now also J21.1 (Pin_1)
- net BUTTON: no longer U2.24 (17_A3_TX4_SDA1)
- net GND: now also J21.7 (Pin_7)
- net SPEAKER: no longer U2.20 (13_SCK_CRX1_LED)
- net VSENSE: no longer U2.28 (21_A7_RX5_BCLK1)
- net INT1: now reaches U2.27 (20_A6_TX5_LRCLK1)
- net INT1: now also J21.6 (Pin_6)
- net MPU6050_SDA renamed GPIO1
- net PB3_1 renamed CS
- net CS: now also J21.5 (Pin_5); no longer MESC1.6 (Pin_6)
- net PB4_1 renamed GPIO3
- net GPIO3: no longer U2.13 (11_MOSI_CTX1)
- net PB4_2 renamed GPIO4
- net GPIO4: now also MESC1.6 (Pin_6)
- net PB5_1 renamed GPIO2
- net GPIO2: now also U2.24 (17_A3_TX4_SDA1); no longer U2.14 (12_MISO_MQSL)
- new net MISO: J21.2 (Pin_2), U2.14 (12_MISO_MQSL)
- new net MOSI: J21.4 (Pin_4), U2.13 (11_MOSI_CTX1)
- new net SCLK: J21.3 (Pin_3), U2.20 (13_SCK_CRX1_LED)

Commit message: documentation stuff
Changed lines of the file:
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@@
 	(wire
 		(pts
-			(xy 149.86 100.965) (xy 134.62 100.965)
+			(xy 43.18 92.71) (xy 43.18 97.79)
 		)
 		(stroke
@@
 	(wire
 		(pts
-			(xy 43.18 92.71) (xy 43.18 97.79)
+			(xy 52.07 53.34) (xy 49.53 53.34)
 		)
 		(stroke
@@
 	(wire
 		(pts
-			(xy 52.07 53.34) (xy 49.53 53.34)
+			(xy 238.76 80.01) (xy 226.06 80.01)
 		)
 		(stroke
@@
 		)
 	)
-	(wire
-		(pts
-			(xy 238.76 80.01) (xy 226.06 80.01)
-		)
-		(stroke
-			(width 0)
-			(type default)
-		)
-	)
 	(text "Teensy 4.0/4.1\nESP32\nUART\nRC receiver connector (for PWM/PPM/SBUS input)\nOptional UART debug header\nOptional I²C header (for sensors like INA219 or IMU)\nPower input connector\nVoltage divider (to monitor battery voltage)\nPush-button E-stop connector\nPower button (for system on/off)\nIMU connector (e.g., MPU-6050 or BNO085)\nencoder inputs (if reading position directly)\nbuzzer (for system alerts or E-stop signal)\nSWD debug access for Teensy\n"
 		(exclude_from_sim no)
@@
 	(label "LED2"
 		(at 147.32 97.79 180)
+		(fields_autoplaced yes)
 		(effects
 			(font
@@
 	(label "ESP_RX"
 		(at 154.94 21.59 0)
+		(fields_autoplaced yes)
 		(effects
 			(font
@@
 	(label "CAN_RX"
 		(at 238.76 85.09 180)
+		(fields_autoplaced yes)
 		(effects
 			(font
@@
 	(label "GND"
 		(at 238.76 80.01 180)
+		(fields_autoplaced yes)
 		(effects
 			(font
@@
 	(label "SPEAKER"
 		(at 154.94 69.85 0)
+		(fields_autoplaced yes)
 		(effects
 			(font
@@
 	(label "ESP_RX"
 		(at 147.32 83.82 180)
+		(fields_autoplaced yes)
 		(effects
 			(font
@@
 	(label "GPIO2"
 		(at 154.94 77.47 0)
+		(fields_autoplaced yes)
 		(effects
 			(font
@@
 	(label "MISO"
 		(at 154.94 52.07 0)
+		(fields_autoplaced yes)
 		(effects
 			(font
@@
 	(label "CAN_TX"
 		(at 238.76 87.63 180)
+		(fields_autoplaced yes)
 		(effects
 			(font
@@
 	(label "GPIO1"
 		(at 154.94 80.01 0)
+		(fields_autoplaced yes)
 		(effects
 			(font
@@
 	(label "GND"
 		(at 154.94 19.05 0)
+		(fields_autoplaced yes)
 		(effects
 			(font
@@
 	(label "CS"
 		(at 154.94 46.99 0)
+		(fields_autoplaced yes)
 		(effects
 			(font
@@
 	(label "RC_Steering"
 		(at 154.94 44.45 0)
+		(fields_autoplaced yes)
 		(effects
 			(font
@@
 	(label "GND"
 		(at 154.94 59.69 0)
+		(fields_autoplaced yes)
 		(effects
 			(font
@@
 	(label "ESP_TX"
 		(at 154.94 24.13 0)
+		(fields_autoplaced yes)
 		(effects
 			(font
@@
 	(label "INT1"
 		(at 154.94 85.09 0)
+		(fields_autoplaced yes)
 		(effects
 			(font
@@
 	(label "CAN_RX"
 		(at 26.67 63.5 0)
+		(fields_autoplaced yes)
 		(effects
 			(font
@@
 	(label "GPIO4"
 		(at 154.94 72.39 0)
+		(fields_autoplaced yes)
 		(effects
 			(font
@@
 	(label "LED2"
 		(at 154.94 29.21 0)
-		(effects
-			(font
-				(size 1.27 1.27)
-			)
-			(justify left bottom)
-		)
-	)
-	(label "VSENSE"
-		(at 149.86 100.965 180)
-		(effects
-			(font
-				(size 1.27 1.27)
-			)
-			(justify right bottom)
+		(fields_autoplaced yes)
+		(effects
+			(font
+				(size 1.27 1.27)
+			)
+			(justify left bottom)
 		)
 	)
 	(label "+5V"
 		(at 238.76 77.47 180)
+		(fields_autoplaced yes)
 		(effects
 			(font
@@
 	(label "RC_Mode"
 		(at 154.94 39.37 0)
+		(fields_autoplaced yes)
 		(effects
 			(font
@@
 	(label "BUTTON"
 		(at 154.94 82.55 0)
+		(fields_autoplaced yes)
 		(effects
 			(font
@@
 	(label "RC_Throttle"
 		(at 154.94 41.91 0)
+		(fields_autoplaced yes)
 		(effects
 			(font
@@
 	(label "MOSI"
 		(at 154.94 49.53 0)
+		(fields_autoplaced yes)
 		(effects
 			(font
@@
 	(label "LED1"
 		(at 147.32 95.25 180)
+		(fields_autoplaced yes)
 		(effects
 			(font
@@
 	(label "SCLK"
 		(at 154.94 67.31 0)
+		(fields_autoplaced yes)
 		(effects
 			(font
@@
 	(label "CAN_TX"
 		(at 26.67 60.96 0)
+		(fields_autoplaced yes)
 		(effects
 			(font
@@
 	(label "LED1"
 		(at 154.94 26.67 0)
+		(fields_autoplaced yes)
 		(effects
 			(font
@@
 	(label "GPIO3"
 		(at 154.94 74.93 0)
+		(fields_autoplaced yes)
 		(effects
 			(font
@@
 	(label "ESP_TX"
 		(at 147.32 86.36 180)
+		(fields_autoplaced yes)
 		(effects
 			(font
@@
 				(hide yes)
 			)
-		)
-	)
-	(global_label "VSENSE"
-		(shape input)
-		(at 134.62 100.965 180)
-		(fields_autoplaced yes)
-		(effects
-			(font
-				(size 1.27 1.27)
-			)
-			(justify right)
-		)
-		(property "Intersheetrefs" "${INTERSHEET_REFS}"
-			(at 124.4987 100.965 0)
-			(effects
-				(font
-					(size 1.27 1.27)
-				)
-				(justify right)
-				(hide yes)
-			)

Commit message: BLDC inductance measurement
Parts:
- renumbered R3 to 10k_1, J2 to CAN1, R7 to R_120, U2 to U1
Changed lines of the file:
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@@
 (kicad_sch
-	(version 20231120)
+	(version 20250114)
 	(generator "eeschema")
-	(generator_version "8.0")
+	(generator_version "9.0")
 	(paper "User" 254 177.8)
+	(text "Teensy 4.0/4.1\nESP32\nUART\nRC receiver connector (for PWM/PPM/SBUS input)\nOptional UART debug header\nOptional I²C header (for sensors like INA219 or IMU)\nPower input connector\nVoltage divider (to monitor battery voltage)\nPush-button E-stop connector\nPower button (for system on/off)\nIMU connector (e.g., MPU-6050 or BNO085)\nencoder inputs (if reading position directly)\nbuzzer (for system alerts or E-stop signal)\nSWD debug access for Teensy\n"
+		(exclude_from_sim no)
+		(at 165.1 109.728 0)
+		(effects
+			(font
+				(face "Courier")
+				(size 1.524 1.524)
+			)
+			(justify left)
+		)
+	)
+	(text "MP2 SER"
+		(exclude_from_sim no)
+		(at 34.29 38.1 0)
+		(effects
+			(font
+				(size 1.2 1.2)
+			)
+			(justify left bottom)
+		)
+	)
+	(text "MESC I/O\nReserved 2 GPIO pins on Teensy for emergency shutoff to MESC\nCAN connector (for MESC motor control)\nVoltage divider (to monitor battery voltage)\n\n"
+		(exclude_from_sim no)
+		(at 165.1 137.414 0)
+		(effects
+			(font
+				(face "Courier")
+				(size 1.4986 1.4986)
+			)
+			(justify left)
+		)
+	)
+	(text "3.3V CAN transcievers only"
+		(exclude_from_sim no)
+		(at 52.07 73.66 0)
+		(effects
+			(font
+				(size 1.27 1.27)
+			)
+		)
+	)
+	(text "Not great design w/ DC-DC conversion from high voltage VBat "
+		(exclude_from_sim no)
+		(at 184.404 144.526 0)
+		(effects
+			(font
+				(size 1.27 1.27)
+			)
+		)
+	)
 	(junction
 		(at 90.17 31.75)
@@
 		)
 	)
-	(text "Teensy 4.0/4.1\nESP32\nUART\nRC receiver connector (for PWM/PPM/SBUS input)\nOptional UART debug header\nOptional I²C header (for sensors like INA219 or IMU)\nPower input connector\nVoltage divider (to monitor battery voltage)\nPush-button E-stop connector\nPower button (for system on/off)\nIMU connector (e.g., MPU-6050 or BNO085)\nencoder inputs (if reading position directly)\nbuzzer (for system alerts or E-stop signal)\nSWD debug access for Teensy\n"
-		(exclude_from_sim no)
-		(at 165.1 109.728 0)
-		(effects
-			(font
-				(face "Courier")
-				(size 1.524 1.524)
-			)
-			(justify left)
-		)
-	)
-	(text "MP2 SER"
-		(exclude_from_sim no)
-		(at 34.29 38.1 0)
-		(effects
-			(font
-				(size 1.2 1.2)
-			)
-			(justify left bottom)
-		)
-	)
-	(text "MESC I/O\nReserved 2 GPIO pins on Teensy for emergency shutoff to MESC\nCAN connector (for MESC motor control)\nVoltage divider (to monitor battery voltage)\n\n"
-		(exclude_from_sim no)
-		(at 165.1 137.414 0)
-		(effects
-			(font
-				(face "Courier")
-				(size 1.4986 1.4986)
-			)
-			(justify left)
-		)
-	)
-	(text "3.3V CAN transcievers only"
-		(exclude_from_sim no)
-		(at 52.07 73.66 0)
-		(effects
-			(font
-				(size 1.27 1.27)
-			)
-		)
-	)
-	(text "Not great design w/ DC-DC conversion from high voltage VBat "
-		(exclude_from_sim no)
-		(at 184.404 144.526 0)
-		(effects
-			(font
-				(size 1.27 1.27)
-			)
-		)
-	)
 	(label "LED2"
 		(at 147.32 97.79 180)
-		(fields_autoplaced yes)
 		(effects
 			(font
@@
 	(label "ESP_RX"
 		(at 154.94 21.59 0)
-		(fields_autoplaced yes)
 		(effects
 			(font
@@
 	(label "CAN_RX"
 		(at 238.76 85.09 180)
-		(fields_autoplaced yes)
 		(effects
 			(font
@@
 	(label "GND"
 		(at 238.76 80.01 180)
-		(fields_autoplaced yes)
 		(effects
 			(font
@@
 	(label "SPEAKER"
 		(at 154.94 69.85 0)
-		(fields_autoplaced yes)
 		(effects
 			(font
@@
 	(label "ESP_RX"
 		(at 147.32 83.82 180)
-		(fields_autoplaced yes)
 		(effects
 			(font
@@
 	(label "GPIO2"
 		(at 154.94 77.47 0)
-		(fields_autoplaced yes)
 		(effects
 			(font
@@
 	(label "MISO"
 		(at 154.94 52.07 0)
-		(fields_autoplaced yes)
 		(effects
 			(font
@@
 	(label "CAN_TX"
 		(at 238.76 87.63 180)
-		(fields_autoplaced yes)
 		(effects
 			(font
@@
 	(label "GPIO1"
 		(at 154.94 80.01 0)
-		(fields_autoplaced yes)
 		(effects
 			(font
@@
 	(label "GND"
 		(at 154.94 19.05 0)
-		(fields_autoplaced yes)
 		(effects
 			(font
@@
 	(label "CS"
 		(at 154.94 46.99 0)
-		(fields_autoplaced yes)
 		(effects
 			(font
@@
 	(label "RC_Steering"
 		(at 154.94 44.45 0)
-		(fields_autoplaced yes)
 		(effects
 			(font
@@
 	(label "GND"
 		(at 154.94 59.69 0)
-		(fields_autoplaced yes)
 		(effects
 			(font
@@
 	(label "ESP_TX"
 		(at 154.94 24.13 0)
-		(fields_autoplaced yes)
 		(effects
 			(font
@@
 	(label "INT1"
 		(at 154.94 85.09 0)
-		(fields_autoplaced yes)
 		(effects
 			(font
@@
 	(label "CAN_RX"
 		(at 26.67 63.5 0)
-		(fields_autoplaced yes)
 		(effects
 			(font
@@
 	(label "GPIO4"
 		(at 154.94 72.39 0)
-		(fields_autoplaced yes)
 		(effects
 			(font
@@
 	(label "LED2"
 		(at 154.94 29.21 0)
-		(fields_autoplaced yes)
 		(effects
 			(font
@@
 	(label "+5V"
 		(at 238.76 77.47 180)
-		(fields_autoplaced yes)
 		(effects
 			(font
@@
 	(label "RC_Mode"
 		(at 154.94 39.37 0)
-		(fields_autoplaced yes)
 		(effects
 			(font
@@
 	(label "BUTTON"
 		(at 154.94 82.55 0)
-		(fields_autoplaced yes)
 		(effects
 			(font
@@
 	(label "RC_Throttle"
 		(at 154.94 41.91 0)
-		(fields_autoplaced yes)
 		(effects
 			(font
@@
 	(label "MOSI"
 		(at 154.94 49.53 0)
-		(fields_autoplaced yes)
 		(effects
 			(font
@@
 	(label "LED1"
 		(at 147.32 95.25 180)
-		(fields_autoplaced yes)
 		(effects
 			(font
@@
 	(label "SCLK"
 		(at 154.94 67.31 0)
-		(fields_autoplaced yes)
 		(effects
 			(font
@@
 	(label "CAN_TX"
 		(at 26.67 60.96 0)
-		(fields_autoplaced yes)
 		(effects
 			(font
@@
 	(label "LED1"
 		(at 154.94 26.67 0)
-		(fields_autoplaced yes)
 		(effects
 			(font
@@
 	(label "GPIO3"
 		(at 154.94 74.93 0)
-		(fields_autoplaced yes)
 		(effects
 			(font
@@
 	(label "ESP_TX"
 		(at 147.32 86.36 180)
-		(fields_autoplaced yes)
 		(effects
 			(font
@@
 		(dnp no)
 		(fields_autoplaced yes)
-		(property "Reference" "R7"
+		(property "Reference" "R_120"
 			(at 67.31 66.675 0)
 			(effects
@@
 		(on_board yes)
 		(dnp no)
-		(property "Reference" "R3"
+		(property "Reference" "10k_1"
 			(at 32.385 74.93 0)
 			(effects
@@
 		(on_board yes)
 		(dnp no)
-		(property "Reference" "U2"
+		(property "Reference" "U1"
 			(at 44.45 55.88 0)
 			(effects
@@
 		(dnp no)
 		(fields_autoplaced yes)
-		(property "Reference" "J2"
+		(property "Reference" "CAN1"
 			(at 36.83 38.1 0)
 			(effects
@@
 		(at 128.27 19.05)
 		(size 17.78 22.86)
+		(exclude_from_sim no)
+		(in_bom yes)
+		(on_board yes)
+		(dnp no)
 		(fields_autoplaced yes)
 		(stroke
@@
 		(at 101.6 19.05)
 		(size 19.05 22.86)
+		(exclude_from_sim no)
+		(in_bom yes)
+		(on_board yes)
+		(dnp no)
 		(fields_autoplaced yes)
 		(stroke
@@
 		)
 	)
+	(embedded_fonts no)
 )
