File: brainboardV1.2/POWER.kicad_sch (KiCad schematic)
At the start: 21 parts, among them J22 Conn_01x01, J24 Conn_01x01, J25 Conn_01x01, U23 PQDE6W-Q110 / RD5-110S12W, U24 12_DCDC_5

Commit message: finalizing brain board v1.2
Parts:
- removed 20k_3: 20k, Resistor_SMD:R_0603_1608Metric, symbol Device:R
- removed C23: 100nF, Capacitor_SMD:C_0805_2012Metric, symbol Device:C
- removed C24, C26, C28, C29: 10uF, Capacitor_SMD:C_0603_1608Metric, symbol Device:C
- removed D23: BZG03C15, Diode_SMD:D_SMA, symbol Diode:SM6T75A
- removed D_BLU1: LED BLU, LED_SMD:LED_0603_1608Metric, symbol Device:LED
- removed SW_SPDT21: SW_SPDT, Button_Switch_THT:SW_NKK_BB15AH, symbol Switch:SW_SPDT
- removed Tp12V21: 12V Pad, TestPoint:TestPoint_THTPad_D2.0mm_Drill1.0mm, symbol Connector:TestPoint
- removed U23: PQDE6W-Q110 / RD5-110S12W, MP2_DFN_Custom_parts:PQDE6W, symbol MP2_DFN_Custom_Symbols:PQDE6W-Q110
- added 20k_21: 20k, Resistor_SMD:R_0603_1608Metric, symbol Device:R
- added C21: 100nF, Capacitor_SMD:C_0805_2012Metric, symbol Device:C
- added C23: C_Polarized_Small_US, Capacitor_Tantalum_SMD:CP_EIA-3216-18_Kemet-A, symbol Device:C_Polarized_Small_US
- added D_BLU21: LED BLU, LED_SMD:LED_0603_1608Metric, symbol Device:LED
- added U21: LD1117S18TR_SOT223, Package_TO_SOT_SMD:SOT-223-3_TabPin2, symbol Regulator_Linear:LD1117S18TR_SOT223
- C25, C27: footprint Capacitor_SMD:C_0603_1608Metric -> Capacitor_SMD:C_0805_2012Metric
Connections:
- net +12V is gone; now on net Vcc: U24.1 (VIN)
- net +3.3V: now also C23.1, D_BLU21.2 (A), U21.2 (VO)
- net +5V: now also U21.3 (VI)
- net GND: now also 20k_21.1, C21.2, C23.2, U21.1 (GND)
- net Vcc: now also C21.1
- new net: 20k_21.2, D_BLU21.1 (K)
Other:
- moved on the sheet: C25, C27, U24

Commit message: documentation stuff
Parts:
- added J23: Conn_01x01, Connector_PinSocket_2.54mm:PinSocket_1x01_P2.54mm_Vertical, symbol Connector_Generic:Conn_01x01
Connections:
- net +5V: now also J23.1 (Pin_1)
Other:
- moved on the sheet: 20k_1, 5k_2, D_GRN1, D_RED1

Commit message: BLDC inductance measurement
Changed lines of the file:
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@@
 (kicad_sch
-	(version 20231120)
+	(version 20250114)
 	(generator "eeschema")
-	(generator_version "8.0")
+	(generator_version "9.0")
 	(paper "A4")
 	(junction
